File: Room Sensor.kicad_pcb (KiCad board)
At the start: 2 copper layers, 70 x 100 mm, 15 parts, among them SW1 SW_Push, SW2 SW_Push, SW3 SW_Push, SW4 SW_Push, U2 ESP32-C3_SUPERMINI_TH

Commit message: Add KiCad latching USB power interface
Parts:
- added J_PWR: USB5V_SW_COM_SW_NO_GND, PinHeader_1x04_P2.54mm_Vertical, B.Cu at (110.0, 145.0)
Routing:
- net /GND: track 319.2 -> 340.4 mm
- net /VIN (5.0v): track 105.3 -> 121.0 mm
- net /USB_VBUS_RAW: track 0.00 -> 2.54 mm

Commit message: Add board-mounted USB-C power input
Parts:
- added J_USB: GCT USB4125-03-C USB-C Power Input, USB_C_Receptacle_GCT_USB4125-xx-x_6P_TopMnt_Horizontal, B.Cu at (121.0, 146.1)
- added R_CC1: 5.1k, R_0805_2012Metric, B.Cu at (125.0, 139.8)
- added R_CC2: 5.1k, R_0805_2012Metric, B.Cu at (117.0, 139.8)
- moved J_PWR 12.3 mm to (104.5, 134.0), turned to 0 degrees
Routing:
- net /GND: track 340.4 -> 387.1 mm, vias 1 -> 3
- net /USB_VBUS_RAW: track 2.54 -> 29.2 mm, vias 0 -> 2
- net /VIN (5.0v): track 121.0 -> 144.4 mm, vias 1 -> 3
- net /BTN_DOWN: track 150.3 -> 156.2 mm
- net /USB_CC2: track 0.00 -> 5.64 mm
- net /USB_CC1: track 0.00 -> 5.64 mm
- net /BTN_SELECT: track 152.4 -> 149.7 mm, vias 0 -> 2

Commit message: Complete PCB manufacturing audit
Parts:
- J_USB: value GCT USB4125-03-C USB-C Power Input -> GCT USB4125-GF-A (1.00 mm shell stake)
Routing:
- net /CS: vias 2 -> 1
Changed lines of the file:
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@@
 			)
 		)
-		(property "Value" "GCT USB4125-03-C USB-C Power Input"
+		(property "Value" "GCT USB4125-GF-A (1.00 mm shell stake)"
 			(at 0 -4.725 0)
 			(unlocked yes)
@@
 	)
 	(via
-		(at 135.12 66)
-		(size 1)
-		(drill 0.5)
-		(layers "F.Cu" "B.Cu")
-		(net "/CS")
-	)
-	(via
 		(at 149 80)
 		(size 1)
@@
 	)
 	(segment
+		(start 121.5 140)
+		(end 124.0875 139.8)
+		(width 0.25)
+		(layer "B.Cu")
+		(net "/USB_CC1")
+	)
+	(segment
+		(start 121.5 143.045)
+		(end 121.5 140)
+		(width 0.25)
+		(layer "B.Cu")
+		(net "/USB_CC1")
+	)
+	(segment
 		(start 118.8 141.2)
 		(end 119 138)
@@
 	)
 	(segment
-		(start 121.5 140)
-		(end 124.0875 139.8)
-		(width 0.25)
-		(layer "B.Cu")
-		(net "/USB_CC1")
-	)
-	(segment
-		(start 121.5 143.045)
-		(end 121.5 140)
-		(width 0.25)
-		(layer "B.Cu")
-		(net "/USB_CC1")
-	)
-	(segment
